File: dru/JLPCB-2Layer/JLCPCB.kicad_pcb (KiCad board)
At the start: 4 copper layers, 180 x 235 mm, 27 parts

Commit message: dru updates
Routing:
- net GND: track 694.5 -> 624.9 mm
- net +5V: track 424.8 -> 416.0 mm
Other:
- copper layers 4 -> 2
Changed lines of the file:
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@@
   (layers
     (0 "F.Cu" signal)
-    (1 "In1.Cu" signal)
-    (2 "In2.Cu" signal)
     (31 "B.Cu" signal)
     (32 "B.Adhes" user "B.Adhesive")
@@
       (layer "F.Mask" (type "Top Solder Mask") (thickness 0.01))
       (layer "F.Cu" (type "copper") (thickness 0.035))
-      (layer "dielectric 1" (type "prepreg") (thickness 0.1) (material "FR4") (epsilon_r 4.5) (loss_tangent 0.02))
-      (layer "In1.Cu" (type "copper") (thickness 0.035))
-      (layer "dielectric 2" (type "core") (thickness 1.24) (material "FR4") (epsilon_r 4.5) (loss_tangent 0.02))
-      (layer "In2.Cu" (type "copper") (thickness 0.035))
-      (layer "dielectric 3" (type "prepreg") (thickness 0.1) (material "FR4") (epsilon_r 4.5) (loss_tangent 0.02))
+      (layer "dielectric 1" (type "core") (thickness 1.51) (material "FR4") (epsilon_r 4.5) (loss_tangent 0.02))
       (layer "B.Cu" (type "copper") (thickness 0.035))
       (layer "B.Mask" (type "Bottom Solder Mask") (thickness 0.01))
@@
         (effects (font (size 1 1) (thickness 0.15)))
     )
-    (pad "" np_thru_hole circle (at 0 0) (size 1.2 1.2) (drill 1) (layers "F&B.Cu" "*.Mask"))
+    (pad "" np_thru_hole circle (at 0 0) (size 1.2 1.2) (drill 1) (layers "*.Cu" "*.Mask"))
     (model "${KICAD6_3DMODEL_DIR}/Connector_Pin.3dshapes/Pin_D0.7mm_L6.5mm_W1.8mm_FlatFork.wrl"
       (offset (xyz 0 0 0))
@@
         (effects (font (size 1 1) (thickness 0.15)))
     )
-    (pad "" np_thru_hole circle (at 0 0) (size 1 1) (drill 0.45) (layers "F&B.Cu" "*.Mask"))
+    (pad "" np_thru_hole circle (at 0 0) (size 1 1) (drill 0.45) (layers "*.Cu" "*.Mask"))
   )
   (footprint "Resistor_SMD:R_0805_2012Metric" (layer "F.Cu")
@@
         (effects (font (size 1 1) (thickness 0.15)))
     )
-    (pad "" np_thru_hole circle (at 0 0) (size 1.2 1.2) (drill 1) (layers "F&B.Cu" "*.Mask"))
+    (pad "" np_thru_hole circle (at 0 0) (size 1.2 1.2) (drill 1) (layers "*.Cu" "*.Mask"))
     (model "${KICAD6_3DMODEL_DIR}/Connector_Pin.3dshapes/Pin_D0.7mm_L6.5mm_W1.8mm_FlatFork.wrl"
       (offset (xyz 0 0 0))
@@
         (effects (font (size 1 1) (thickness 0.15)))
     )
-    (pad "" np_thru_hole circle (at 0 0) (size 1 1) (drill 0.55) (layers "F&B.Cu" "*.Mask"))
+    (pad "" np_thru_hole circle (at 0 0) (size 1 1) (drill 0.55) (layers "*.Cu" "*.Mask"))
   )
   (footprint "MountingHole:MountingHole_2.2mm_M2_DIN965_Pad_TopBottom" (layer "F.Cu")
@@
   (via (at 141.8 139) (size 0.55) (drill 0.4) (layers "F.Cu" "B.Cu") (net 1))
   (via (at 137 189) (size 0.8) (drill 0.4) (layers "F.Cu" "B.Cu") (net 1))
-  (segment (start 135 50.993407) (end 136.444 49.349407) (width 0.25) (layer "In1.Cu") (net 1))
-  (segment (start 134 50.993407) (end 135 50.993407) (width 0.25) (layer "In1.Cu") (net 1))
-  (segment (start 130.706045 50.993407) (end 129.079835 49.293407) (width 0.25) (layer "In1.Cu") (net 1))
-  (segment (start 134 50.993407) (end 130.706045 50.993407) (width 0.25) (layer "In1.Cu") (net 1))
   (segment (start 132 52) (end 131 53) (width 0.25) (layer "B.Cu") (net 1))
   (segment (start 143 172) (end 143 169.9) (width 0.25) (layer "B.Cu") (net 1))
@@
   (via (at 132 48.993407) (size 0.8) (drill 0.4) (layers "F.Cu" "B.Cu") (net 2))
   (via (at 121 129) (size 0.5) (drill 0.4) (layers "F.Cu" "B.Cu") (net 2))
-  (segment (start 115 41) (end 132 41) (width 0.08) (layer "In1.Cu") (net 2))
-  (segment (start 132 48.993407) (end 149.6408 48.993407) (width 0.25) (layer "In1.Cu") (net 2))
-  (segment (start 131.991304 48.984711) (end 115.008696 48.984711) (width 0.25) (layer "In1.Cu") (net 2))
-  (segment (start 132 41) (end 150 41) (width 0.1) (layer "In1.Cu") (net 2))
   (segment (start 132 33) (end 131.991304 32.991304) (width 0.25) (layer "B.Cu") (net 2))
   (group "" (id 52a65b04-d1e9-4539-8de9-564f6660c319)
